File: display.brd (EAGLE design)
At the start: 100 x 80 mm, 70 parts, among them IC1 74595, IC2 74595, IC3 74595, IC4 74595

Commit message: Renamed controller > display. Removed resitor names. Added IC1 QH to IC2 serial.
Parts:
- moved IC1 63.2 mm to (27.9, 19.1), turned to 180 degrees
- moved IC3 63.2 mm to (86.4, 43.2), turned to 270 degrees
Connections:
- removed net SERIAL1: IC1.14, IC2.9
- new net SERIAL3: IC2.9, IC3.14
- net N$14: now also IC3.15; no longer IC1.15
- net N$31: now also IC3.1; no longer IC1.1
- net N$32: now also IC3.2; no longer IC1.2
- net N$33: now also IC3.3; no longer IC1.3
- net N$34: now also IC3.4; no longer IC1.4
- net N$35: now also IC3.5; no longer IC1.5
- net N$36: now also IC3.6; no longer IC1.6
- net N$37: now also IC3.7; no longer IC1.7
- net N$49: now also IC1.7; no longer IC3.7
- net N$50: now also IC1.6; no longer IC3.6
- net N$52: now also IC1.4; no longer IC3.4
- net N$53: now also IC1.3; no longer IC3.3
- net N$54: now also IC1.2; no longer IC3.2
- net N$63: now also IC1.5; no longer IC3.5
- net SERIAL2: now also IC1.9; no longer IC3.9
- net SERIAL4: now also IC3.9; no longer IC1.9
- net SERIALIN: now also IC1.14; no longer IC3.14
Routing:
- net SERIAL2: track 0.00 -> 69.5 mm, vias 0 -> 2
- net SERIAL1: track 32.3 -> 0.00 mm, vias 2 -> 0
- net SERIAL3: track 0.00 -> 30.4 mm, vias 0 -> 2
- net GND: track 235.7 -> 232.1 mm

Commit message: Beginning of new controller board layout.
Parts:
- added FRAME1: FRAME-LETTER, SparkFun-Aesthetics:CREATIVE_COMMONS
Changed lines of the file:
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@@
 <element name="C3" library="SparkFun-Passives" package="0805" value="" x="88.9" y="48.26" rot="R270"/>
 <element name="C4" library="SparkFun-Passives" package="0805" value="" x="13.97" y="44.45" rot="R90"/>
+<element name="FRAME1" library="SparkFun-Aesthetics" package="CREATIVE_COMMONS" value="FRAME-LETTER" x="11.43" y="-12.7"/>
 </elements>
 <signals>
