File: snoozerly.sch (EAGLE design)
At the start: 55 parts, among them Q1 MOSFET_PCHANNEL, Q2 MOSFET-NCHANNELFDD8780, Q3 MOSFET-NCHANNELBSS123LT1G, Q4 MOSFET-NCHANNELBSS123LT1G, U1 ATMEGA328P, Y1 32KHz, Y2 8MHz

Commit message: Merge branch 'master' into rev-0.1
Connections:
- net PWM_LED renamed PWM_STRIP
Other:
- moved on the sheet: LED1, LED2, LED3, LED4, LED5, LED6, LED7, LEDSTRIP, NOKIA5110, Q2, Q3, Q4

Commit message: fixed touch sensor vcc and gnd. increased docu fonts.
Connections:
- net 5V: now also AT42QT1070.VDD; no longer AT42QT1070.VSS
- net GND: now also AT42QT1070.VSS; no longer AT42QT1070.VDD
Changed lines of the file:
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@@
 <setting verticaltext="up"/>
 </settings>
-<grid distance="0.1" unitdist="inch" unit="inch" style="lines" multiple="1" display="no" altdistance="0.01" altunitdist="inch" altunit="inch"/>
+<grid distance="0.05" unitdist="inch" unit="inch" style="lines" multiple="1" display="no" altdistance="0.01" altunitdist="inch" altunit="inch"/>
 <layers>
 <layer number="1" name="Top" color="4" fill="1" visible="no" active="no"/>
@@
 <attribute name="VALUE" x="48.26" y="214.63" size="1.778" layer="96"/>
 </instance>
-<instance part="SUPPLY2" gate="1" x="81.28" y="240.03" smashed="yes">
-<attribute name="VALUE" x="80.264" y="237.744" size="1.778" layer="96" rot="R90"/>
-</instance>
-<instance part="GND3" gate="1" x="36.83" y="234.95" smashed="yes" rot="R270">
-<attribute name="VALUE" x="34.29" y="237.49" size="1.778" layer="96" rot="R270"/>
+<instance part="SUPPLY2" gate="1" x="36.83" y="234.95" smashed="yes" rot="R90">
+<attribute name="VALUE" x="39.116" y="233.934" size="1.778" layer="96" rot="R180"/>
+</instance>
+<instance part="GND3" gate="1" x="81.28" y="242.57" smashed="yes" rot="R180">
+<attribute name="VALUE" x="83.82" y="245.11" size="1.778" layer="96" rot="R180"/>
 </instance>
 <instance part="U$7" gate="G$1" x="92.71" y="240.03" smashed="yes">
@@
 </segment>
 <segment>
-<pinref part="AT42QT1070" gate="G$1" pin="VDD"/>
-<wire x1="43.18" y1="234.95" x2="39.37" y2="234.95" width="0.1524" layer="91"/>
-<pinref part="GND3" gate="1" pin="GND"/>
-</segment>
-<segment>
 <pinref part="GND11" gate="1" pin="GND"/>
 <pinref part="NOKIA5110" gate="G$1" pin="/SCE"/>
@@
 <wire x1="134.62" y1="149.86" x2="143.51" y2="149.86" width="0.1524" layer="91"/>
 <label x="135.89" y="149.86" size="1.778" layer="95"/>
+</segment>
+<segment>
+<pinref part="AT42QT1070" gate="G$1" pin="VSS"/>
+<wire x1="78.74" y1="234.95" x2="81.28" y2="234.95" width="0.1524" layer="91"/>
+<pinref part="GND3" gate="1" pin="GND"/>
+<wire x1="81.28" y1="234.95" x2="81.28" y2="240.03" width="0.1524" layer="91"/>
 </segment>
 </net>
@@
 <wire x1="85.09" y1="285.75" x2="85.09" y2="288.29" width="0.1524" layer="91"/>
 <pinref part="5V" gate="1" pin="VCC"/>
-</segment>
-<segment>
-<pinref part="AT42QT1070" gate="G$1" pin="VSS"/>
-<wire x1="78.74" y1="234.95" x2="81.28" y2="234.95" width="0.1524" layer="91"/>
-<wire x1="81.28" y1="234.95" x2="81.28" y2="240.03" width="0.1524" layer="91"/>
-<pinref part="SUPPLY2" gate="1" pin="VCC"/>
 </segment>
 <segment>
@@
 <wire x1="83.82" y1="200.66" x2="88.9" y2="200.66" width="0.1524" layer="91"/>
 </segment>
+<segment>
+<pinref part="SUPPLY2" gate="1" pin="VCC"/>
+<pinref part="AT42QT1070" gate="G$1" pin="VDD"/>
+<wire x1="36.83" y1="234.95" x2="43.18" y2="234.95" width="0.1524" layer="91"/>
+</segment>
 </net>
 <net name="N$1" class="0">
@@
 <pinref part="U$5" gate="G$1" pin="1"/>
 <wire x1="96.52" y1="280.67" x2="96.52" y2="276.86" width="0.1524" layer="91"/>
+<wire x1="96.52" y1="280.67" x2="100.33" y2="280.67" width="0.1524" layer="91"/>
+<junction x="96.52" y="280.67"/>
 </segment>
 <segment>
@@
 <pinref part="U$4" gate="G$1" pin="1"/>
 <wire x1="90.17" y1="278.13" x2="90.17" y2="276.86" width="0.1524" layer="91"/>
-</segment>
-<segment>
+<wire x1="90.17" y1="278.13" x2="92.71" y2="278.13" width="0.1524" layer="91"/>
+<junction x="90.17" y="278.13"/>
+</segment>
+<segment>

Commit message: updates before touch sensor changes.
Parts:
- C1, C2, C3, C6: value 100nF -> 0.1uF
Connections:
- net GND: now also C4.1; no longer U$25.1
- net N$14: now also U$25.2; no longer C4.2
- net N$18: now also C4.2, U$25.1; no longer C4.1, U$25.2
Changed lines of the file:
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@@
 <part name="C5" library="SparkFun-Capacitors" deviceset="CAP_POL" device="C" value="10uF"/>
 <part name="C7" library="SparkFun-Capacitors" deviceset="CAP_POL" device="C" value="10uF"/>
-<part name="C2" library="SparkFun-Capacitors" deviceset="CAP" device="0805" value="100nF"/>
-<part name="C1" library="SparkFun-Capacitors" deviceset="CAP" device="0805" value="100nF"/>
+<part name="C2" library="SparkFun-Capacitors" deviceset="CAP" device="0805" value="0.1uF"/>
+<part name="C1" library="SparkFun-Capacitors" deviceset="CAP" device="0805" value="0.1uF"/>
 <part name="GND8" library="SparkFun-Aesthetics" deviceset="GND" device=""/>
 <part name="GND9" library="SparkFun-Aesthetics" deviceset="GND" device=""/>
@@
 <part name="SUPPLY5" library="SparkFun-Aesthetics" deviceset="VCC" device=""/>
 <part name="GND12" library="SparkFun-Aesthetics" deviceset="GND" device=""/>
-<part name="C3" library="SparkFun-Capacitors" deviceset="CAP" device="0805" value="100nF"/>
+<part name="C3" library="SparkFun-Capacitors" deviceset="CAP" device="0805" value="0.1uF"/>
 <part name="5V" library="SparkFun-Aesthetics" deviceset="VCC" device=""/>
 <part name="SUPPLY7" library="SparkFun-Aesthetics" deviceset="VCC" device=""/>
@@
 <part name="U$16" library="jt_parts" deviceset="RESISTOR" device="" value="100"/>
 <part name="GND11" library="SparkFun-Aesthetics" deviceset="GND" device=""/>
-<part name="C6" library="SparkFun-Capacitors" deviceset="CAP" device="0805" value="100nF"/>
+<part name="C6" library="SparkFun-Capacitors" deviceset="CAP" device="0805" value="0.1uF"/>
 <part name="SUPPLY10" library="SparkFun-Aesthetics" deviceset="VCC" device=""/>
 <part name="SERIAL" library="SparkFun-Connectors" deviceset="M03" device="1X03_NO_SILK"/>
@@
 <attribute name="NAME" x="180.34" y="153.67" size="1.778" layer="95"/>
 </instance>
-<instance part="C4" gate="G$1" x="199.39" y="157.48" smashed="yes" rot="R180">
-<attribute name="VALUE" x="208.534" y="160.401" size="1.778" layer="96" rot="R180"/>
+<instance part="C4" gate="G$1" x="199.39" y="144.78" smashed="yes" rot="R180">
+<attribute name="VALUE" x="208.534" y="147.701" size="1.778" layer="96" rot="R180"/>
 </instance>
 <instance part="U1" gate="G$1" x="68.58" y="151.13" smashed="yes">
@@
 <instance part="GND12" gate="1" x="54.61" y="273.05"/>
 <instance part="C3" gate="G$1" x="67.31" y="264.16" smashed="yes" rot="R270">
-<attribute name="VALUE" x="59.436" y="266.319" size="1.778" layer="96"/>
+<attribute name="VALUE" x="65.786" y="258.699" size="1.778" layer="96"/>
 </instance>
 <instance part="5V" gate="1" x="85.09" y="288.29" smashed="yes">
@@
 <attribute name="VALUE" x="30.226" y="205.486" size="1.778" layer="96" rot="R270"/>
 </instance>
-<instance part="U$25" gate="G$1" x="199.39" y="144.78" smashed="yes" rot="R90">
-<attribute name="VALUE" x="202.692" y="140.97" size="1.778" layer="96" rot="R90"/>
+<instance part="U$25" gate="G$1" x="199.39" y="154.94" smashed="yes" rot="R90">
+<attribute name="VALUE" x="202.692" y="151.13" size="1.778" layer="96" rot="R90"/>
 </instance>
 <instance part="NCP1117" gate="G$1" x="195.58" y="283.21" smashed="yes">
@@
 <wire x1="187.96" y1="151.13" x2="187.96" y2="138.43" width="0.1524" layer="91"/>
 <pinref part="GND6" gate="1" pin="GND"/>
-<pinref part="U$25" gate="G$1" pin="1"/>
 <wire x1="187.96" y1="138.43" x2="184.15" y2="138.43" width="0.1524" layer="91"/>
-<wire x1="199.39" y1="139.7" x2="199.39" y2="138.43" width="0.1524" layer="91"/>
 <wire x1="199.39" y1="138.43" x2="187.96" y2="138.43" width="0.1524" layer="91"/>
 <junction x="187.96" y="138.43"/>
+<pinref part="C4" gate="G$1" pin="1"/>
+<wire x1="199.39" y1="138.43" x2="199.39" y2="139.7" width="0.1524" layer="91"/>
 </segment>
 <segment>
@@
 <pinref part="LEDSTRIP" gate="G$1" pin="2"/>
 <wire x1="198.12" y1="171.45" x2="187.96" y2="171.45" width="0.1524" layer="91"/>
-<pinref part="C4" gate="G$1" pin="2"/>
-<wire x1="199.39" y1="160.02" x2="199.39" y2="162.56" width="0.1524" layer="91"/>
 <wire x1="199.39" y1="162.56" x2="187.96" y2="162.56" width="0.1524" layer="91"/>
 <pinref part="Q2" gate="G$1" pin="D"/>
@@
 <wire x1="187.96" y1="171.45" x2="187.96" y2="162.56" width="0.1524" layer="91"/>
 <junction x="187.96" y="162.56"/>
+<pinref part="U$25" gate="G$1" pin="2"/>
+<wire x1="199.39" y1="160.02" x2="199.39" y2="162.56" width="0.1524" layer="91"/>
 </segment>
 </net>
@@
 </segment>
 </net>
-<net name="N$18" class="0">
-<segment>
-<pinref part="C4" gate="G$1" pin="1"/>
-<pinref part="U$25" gate="G$1" pin="2"/>
-<wire x1="199.39" y1="152.4" x2="199.39" y2="149.86" width="0.1524" layer="91"/>
-</segment>
-</net>
 <net name="PWM_STRIP" class="0">
 <segment>
@@
 </segment>
 </net>
+<net name="N$18" class="0">
+<segment>
+<pinref part="U$25" gate="G$1" pin="1"/>
+<pinref part="C4" gate="G$1" pin="2"/>
+<wire x1="199.39" y1="149.86" x2="199.39" y2="147.32" width="0.1524" layer="91"/>
+</segment>
+</net>

Commit message: increase drill size change remaining.
Parts:
- added C9: 0.1uF, SparkFun-Capacitors:CAP0805
- C1: value 0.1uF -> 100nF
Connections:
- net 5V: now also AT42QT1070.MODE(VDD), AT42QT1070.RESET, C9.1
- net GND: now also C9.2
Changed lines of the file:
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@@
 <part name="C7" library="SparkFun-Capacitors" deviceset="CAP_POL" device="C" value="10uF"/>
 <part name="C2" library="SparkFun-Capacitors" deviceset="CAP" device="0805" value="0.1uF"/>
-<part name="C1" library="SparkFun-Capacitors" deviceset="CAP" device="0805" value="0.1uF"/>
+<part name="C1" library="SparkFun-Capacitors" deviceset="CAP" device="0805" value="100nF"/>
 <part name="GND8" library="SparkFun-Aesthetics" deviceset="GND" device=""/>
 <part name="GND9" library="SparkFun-Aesthetics" deviceset="GND" device=""/>
@@
 <part name="U$25" library="adafruit" deviceset="R-US_" device="R0603" value="zero"/>
 <part name="NCP1117" library="jt_parts" deviceset="VREG-3.3V" device="NCP1117"/>
+<part name="C9" library="SparkFun-Capacitors" deviceset="CAP" device="0805" value="0.1uF"/>
+<part name="GND7" library="SparkFun-Aesthetics" deviceset="GND" device=""/>
 </parts>
 <sheets>
@@
 <attribute name="VALUE" x="48.26" y="214.63" size="1.778" layer="96"/>
 </instance>
-<instance part="SUPPLY2" gate="1" x="36.83" y="234.95" smashed="yes" rot="R90">
-<attribute name="VALUE" x="39.116" y="233.934" size="1.778" layer="96" rot="R180"/>
+<instance part="SUPPLY2" gate="1" x="26.67" y="234.95" smashed="yes" rot="R90">
+<attribute name="VALUE" x="28.956" y="233.934" size="1.778" layer="96" rot="R180"/>
 </instance>
 <instance part="GND3" gate="1" x="81.28" y="242.57" smashed="yes" rot="R180">
@@
 <instance part="NCP1117" gate="G$1" x="195.58" y="283.21" smashed="yes">
 <attribute name="NAME" x="190.5" y="287.02" size="1.778" layer="95"/>
+</instance>
+<instance part="C9" gate="G$1" x="31.75" y="242.57" smashed="yes" rot="R180">
+<attribute name="VALUE" x="26.924" y="241.681" size="1.778" layer="96" rot="R180"/>
+</instance>
+<instance part="GND7" gate="1" x="31.75" y="250.19" smashed="yes" rot="R180">
+<attribute name="VALUE" x="34.29" y="252.73" size="1.778" layer="96" rot="R180"/>
 </instance>
 </instances>
@@
 <pinref part="GND3" gate="1" pin="GND"/>
 <wire x1="81.28" y1="234.95" x2="81.28" y2="240.03" width="0.1524" layer="91"/>
+</segment>
+<segment>
+<pinref part="C9" gate="G$1" pin="2"/>
+<wire x1="31.75" y1="245.11" x2="31.75" y2="246.38" width="0.1524" layer="91"/>
+<wire x1="31.75" y1="247.65" x2="31.75" y2="246.38" width="0.1524" layer="91"/>
+<pinref part="GND7" gate="1" pin="GND"/>
 </segment>
 </net>
@@
 <pinref part="SUPPLY2" gate="1" pin="VCC"/>
 <pinref part="AT42QT1070" gate="G$1" pin="VDD"/>
-<wire x1="36.83" y1="234.95" x2="43.18" y2="234.95" width="0.1524" layer="91"/>
+<wire x1="26.67" y1="234.95" x2="31.75" y2="234.95" width="0.1524" layer="91"/>
+<pinref part="AT42QT1070" gate="G$1" pin="RESET"/>
+<wire x1="31.75" y1="234.95" x2="40.64" y2="234.95" width="0.1524" layer="91"/>
+<wire x1="40.64" y1="234.95" x2="43.18" y2="234.95" width="0.1524" layer="91"/>
+<wire x1="43.18" y1="227.33" x2="40.64" y2="227.33" width="0.1524" layer="91"/>
+<wire x1="40.64" y1="227.33" x2="40.64" y2="232.41" width="0.1524" layer="91"/>
+<junction x="40.64" y="234.95"/>
+<pinref part="AT42QT1070" gate="G$1" pin="MODE(VDD)"/>
+<wire x1="40.64" y1="232.41" x2="40.64" y2="234.95" width="0.1524" layer="91"/>
+<wire x1="43.18" y1="232.41" x2="40.64" y2="232.41" width="0.1524" layer="91"/>
+<junction x="40.64" y="232.41"/>
+<pinref part="C9" gate="G$1" pin="1"/>
+<wire x1="31.75" y1="234.95" x2="31.75" y2="237.49" width="0.1524" layer="91"/>
+<junction x="31.75" y="234.95"/>
 </segment>
 </net>

Commit message: increased 10uf cap pads
Parts:
- C5, C7: device SparkFun-Capacitors:CAP_POLC -> jt_parts:CAP-POLCAP-PANASONIC-C
Changed lines of the file:
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@@
 <setting verticaltext="up"/>
 </settings>
-<grid distance="0.05" unitdist="inch" unit="inch" style="lines" multiple="1" display="no" altdistance="0.01" altunitdist="inch" altunit="inch"/>
+<grid distance="0.1" unitdist="inch" unit="inch" style="lines" multiple="1" display="no" altdistance="0.01" altunitdist="inch" altunit="inch"/>
 <layers>
 <layer number="1" name="Top" color="4" fill="1" visible="no" active="no"/>
@@
 <part name="LED2" library="jt_parts" deviceset="LED" device="" value=""/>
 <part name="LED3" library="jt_parts" deviceset="LED" device="" value=""/>
-<part name="C5" library="SparkFun-Capacitors" deviceset="CAP_POL" device="C" value="10uF"/>
-<part name="C7" library="SparkFun-Capacitors" deviceset="CAP_POL" device="C" value="10uF"/>
+<part name="C5" library="jt_parts" deviceset="CAP-POL" device="CAP-PANASONIC-C" value="10uF"/>
+<part name="C7" library="jt_parts" deviceset="CAP-POL" device="CAP-PANASONIC-C" value="10uF"/>
 <part name="C2" library="SparkFun-Capacitors" deviceset="CAP" device="0805" value="0.1uF"/>
 <part name="C1" library="SparkFun-Capacitors" deviceset="CAP" device="0805" value="100nF"/>
